File: Gra&SP Int Ex/GraSPIntEx.kicad_pcb (KiCad board)
At the start: 2 copper layers, 161.9 x 161.9 mm, 142 parts, among them J1 4P4C, J2 4P4C, SW1 SW_PUSH, SW10 SW_PUSH, SW11 SW_PUSH, SW12 SW_PUSH, SW13 SW_PUSH, SW14 SW_PUSH, SW15 SW_PUSH, SW16 SW_PUSH, SW17 SW_PUSH, SW18 SW_PUSH, SW19 SW_PUSH, SW2 SW_PUSH, SW20 SW_PUSH, SW21 SW_PUSH, SW22 SW_PUSH, SW23 SW_PUSH, SW24 SW_PUSH, SW25 SW_PUSH, SW26 SW_PUSH, SW3 SW_PUSH, SW4 SW_PUSH, SW5 SW_PUSH, SW6 SW_PUSH, SW7 SW_PUSH, SW8 SW_PUSH, SW9 SW_PUSH, U1 Qwiic Pro Micro, U2 Qwiic Pro Micro

Commit message: Printed
Parts:
- renumbered G*** to G1, G*** to G2
