File: Gra&SP Int Ex/GraSPIntTop.kicad_pcb (KiCad board)
At the start: 2 copper layers, 161.9 x 161.9 mm, 26 parts, among them SW1 SW_PUSH, SW10 SW_PUSH, SW11 SW_PUSH, SW12 SW_PUSH, SW13 SW_PUSH, SW14 SW_PUSH, SW15 SW_PUSH, SW16 SW_PUSH, SW17 SW_PUSH, SW18 SW_PUSH, SW19 SW_PUSH, SW2 SW_PUSH, SW20 SW_PUSH, SW21 SW_PUSH, SW22 SW_PUSH, SW23 SW_PUSH, SW24 SW_PUSH, SW25 SW_PUSH, SW26 SW_PUSH, SW3 SW_PUSH, SW4 SW_PUSH, SW5 SW_PUSH, SW6 SW_PUSH, SW7 SW_PUSH, SW8 SW_PUSH, SW9 SW_PUSH

Commit message: Printed
Parts:
- SW1, SW10, SW11, SW12, SW13, SW14, SW15, SW16, SW17, SW18, SW19, SW2, SW20, SW21, SW22, SW23, SW24, SW25, SW26, SW3, SW4, SW5, SW6, SW7, SW8, SW9: footprint kbd:SW_Hole -> my library:SW_Hole
Changed lines of the file:
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@@
     (pcbplotparams
       (layerselection 0x010fc_ffffffff)
-      (usegerberextensions false)
+      (usegerberextensions true)
       (usegerberattributes true)
       (usegerberadvancedattributes true)
@@
       (outputformat 1)
       (mirror false)
-      (drillshape 1)
+      (drillshape 0)
       (scaleselection 1)
       (outputdirectory ""))
@@
     (uvia_drill 0.1)
   )
-  (module kbd:SW_Hole (layer F.Cu)
+  (module "my library:SW_Hole" (layer F.Cu)
     (at 152.4 85.725)
     (fp_text reference SW18 (at 4.6 6 180) (layer Dwgs.User) hide
@@
     (fp_line (start 7 -7) (end -7 -7) (layer Edge.Cuts) (width 0.12))
   )
-  (module kbd:SW_Hole (layer F.Cu)
+  (module "my library:SW_Hole" (layer F.Cu)
     (at 47.625 123.825)
     (fp_text reference SW25 (at 4.6 6 180) (layer Dwgs.User) hide
@@
     (fp_line (start 7 -7) (end -7 -7) (layer Edge.Cuts) (width 0.12))
   )
-  (module kbd:SW_Hole (layer F.Cu)
+  (module "my library:SW_Hole" (layer F.Cu)
     (at 133.35 42.8625)
     (fp_text reference SW5 (at 4.6 6 180) (layer Dwgs.User) hide
@@
     (fp_line (start 7 -7) (end -7 -7) (layer Edge.Cuts) (width 0.12))
   )
-  (module kbd:SW_Hole (layer F.Cu)
+  (module "my library:SW_Hole" (layer F.Cu)
     (at 138.1125 105.592116 315)
     (fp_text reference SW20 (at 4.6 6 315) (layer Dwgs.User) hide
@@
     (fp_line (start 7 -7) (end -7 -7) (layer Edge.Cuts) (width 0.12))
   )
-  (module kbd:SW_Hole (layer F.Cu)
+  (module "my library:SW_Hole" (layer F.Cu)
     (at 152.4 47.625)
     (fp_text reference SW6 (at 4.6 6 180) (layer Dwgs.User) hide
@@
     (fp_line (start 7 -7) (end -7 -7) (layer Edge.Cuts) (width 0.12))
   )
-  (module kbd:SW_Hole (layer F.Cu)
+  (module "my library:SW_Hole" (layer F.Cu)
     (at 133.35 80.9625)
     (fp_text reference SW17 (at 4.6 6 180) (layer Dwgs.User) hide
@@
     (fp_line (start 7 -7) (end -7 -7) (layer Edge.Cuts) (width 0.12))
   )
-  (module kbd:SW_Hole (layer F.Cu)
+  (module "my library:SW_Hole" (layer F.Cu)
     (at 95.25 52.3875)
     (fp_text reference SW9 (at 4.6 6 180) (layer Dwgs.User) hide
@@
     (fp_line (start 7 -7) (end -7 -7) (layer Edge.Cuts) (width 0.12))
   )
-  (module kbd:SW_Hole (layer F.Cu)
+  (module "my library:SW_Hole" (layer F.Cu)
     (at 133.35 61.9125)
     (fp_text reference SW11 (at 4.6 6 180) (layer Dwgs.User) hide
@@
     (fp_line (start 7 -7) (end -7 -7) (layer Edge.Cuts) (width 0.12))
   )
-  (module kbd:SW_Hole (layer F.Cu)
+  (module "my library:SW_Hole" (layer F.Cu)
     (at 76.2 80.9625)
     (fp_text reference SW14 (at 4.6 6 180) (layer Dwgs.User) hide
@@
     (fp_line (start 7 -7) (end -7 -7) (layer Edge.Cuts) (width 0.12))
   )
-  (module kbd:SW_Hole (layer F.Cu)
+  (module "my library:SW_Hole" (layer F.Cu)
     (at 57.15 66.675)
     (fp_text reference SW7 (at 4.6 6 180) (layer Dwgs.User) hide
@@
     (fp_line (start 7 -7) (end -7 -7) (layer Edge.Cuts) (width 0.12))
   )
-  (module kbd:SW_Hole (layer F.Cu)
+  (module "my library:SW_Hole" (layer F.Cu)
     (at 95.25 71.4375)
     (fp_text reference SW15 (at 4.6 6 180) (layer Dwgs.User) hide
@@
     (fp_line (start 7 -7) (end -7 -7) (layer Edge.Cuts) (width 0.12))
   )
-  (module kbd:SW_Hole (layer F.Cu)
+  (module "my library:SW_Hole" (layer F.Cu)
     (at 95.25 33.3375)
     (fp_text reference SW3 (at 4.6 6 180) (layer Dwgs.User) hide
@@
     (fp_line (start 7 -7) (end -7 -7) (layer Edge.Cuts) (width 0.12))
   )
-  (module kbd:SW_Hole (layer F.Cu)
+  (module "my library:SW_Hole" (layer F.Cu)
     (at 114.3 71.4375)
     (fp_text reference SW16 (at 4.6 6 180) (layer Dwgs.User) hide
@@
     (fp_line (start 7 -7) (end -7 -7) (layer Edge.Cuts) (width 0.12))
   )
-  (module kbd:SW_Hole (layer F.Cu)
+  (module "my library:SW_Hole" (layer F.Cu)
     (at 138.1125 132.532884 315)
     (fp_text reference SW23 (at 4.6 6 315) (layer Dwgs.User) hide
@@
     (fp_line (start 7 -7) (end -7 -7) (layer Edge.Cuts) (width 0.12))
   )
-  (module kbd:SW_Hole (layer F.Cu)
+  (module "my library:SW_Hole" (layer F.Cu)
     (at 57.15 85.725)
     (fp_text reference SW13 (at 4.6 6 180) (layer Dwgs.User) hide
@@
     (fp_line (start 7 -7) (end -7 -7) (layer Edge.Cuts) (width 0.12))
   )
-  (module kbd:SW_Hole (layer F.Cu)
+  (module "my library:SW_Hole" (layer F.Cu)
     (at 76.2 42.8625)
     (fp_text reference SW2 (at 4.6 6 180) (layer Dwgs.User) hide
@@
     (fp_line (start 7 -7) (end -7 -7) (layer Edge.Cuts) (width 0.12))
   )
-  (module kbd:SW_Hole (layer F.Cu)
+  (module "my library:SW_Hole" (layer F.Cu)
     (at 114.3 33.3375)
     (fp_text reference SW4 (at 4.6 6 180) (layer Dwgs.User) hide
@@
     (fp_line (start 7 -7) (end -7 -7) (layer Edge.Cuts) (width 0.12))
   )
-  (module kbd:SW_Hole (layer F.Cu)
+  (module "my library:SW_Hole" (layer F.Cu)
     (at 124.642116 119.0625 315)
     (fp_text reference SW21 (at 4.6 6 315) (layer Dwgs.User) hide
@@
     (fp_line (start 7 -7) (end -7 -7) (layer Edge.Cuts) (width 0.12))
   )
-  (module kbd:SW_Hole (layer F.Cu)
+  (module "my library:SW_Hole" (layer F.Cu)
     (at 114.3 52.3875)
     (fp_text reference SW10 (at 4.6 6 180) (layer Dwgs.User) hide
@@
     (fp_line (start 7 -7) (end -7 -7) (layer Edge.Cuts) (width 0.12))
   )
-  (module kbd:SW_Hole (layer F.Cu)
+  (module "my library:SW_Hole" (layer F.Cu)
     (at 76.2 61.9125)
     (fp_text reference SW8 (at 4.6 6 180) (layer Dwgs.User) hide
@@
     (fp_line (start 7 -7) (end -7 -7) (layer Edge.Cuts) (width 0.12))
   )
-  (module kbd:SW_Hole (layer F.Cu)
+  (module "my library:SW_Hole" (layer F.Cu)
     (at 151.582884 119.0625 315)
     (fp_text reference SW22 (at 4.6 6 315) (layer Dwgs.User) hide
@@
     (fp_line (start 7 -7) (end -7 -7) (layer Edge.Cuts) (width 0.12))
   )
-  (module kbd:SW_Hole (layer F.Cu)
+  (module "my library:SW_Hole" (layer F.Cu)
     (at 85.725 152.4)
     (fp_text reference SW26 (at 4.6 6 180) (layer Dwgs.User) hide
@@
     (fp_line (start 7 -7) (end -7 -7) (layer Edge.Cuts) (width 0.12))
   )
-  (module kbd:SW_Hole (layer F.Cu)
+  (module "my library:SW_Hole" (layer F.Cu)
     (at 117.906924 98.856924 315)
     (fp_text reference SW19 (at 4.6 6 315) (layer Dwgs.User) hide
@@
     (fp_line (start 7 -7) (end -7 -7) (layer Edge.Cuts) (width 0.12))
   )
-  (module kbd:SW_Hole (layer F.Cu)
+  (module "my library:SW_Hole" (layer F.Cu)
     (at 152.4 66.675)
     (fp_text reference SW12 (at 4.6 6 180) (layer Dwgs.User) hide
@@
     (fp_line (start 7 -7) (end -7 -7) (layer Edge.Cuts) (width 0.12))
   )
-  (module kbd:SW_Hole (layer F.Cu)
+  (module "my library:SW_Hole" (layer F.Cu)
     (at 158.318076 139.268076 315)
     (fp_text reference SW24 (at 4.6 6 315) (layer Dwgs.User) hide
@@
     (fp_line (start 7 -7) (end -7 -7) (layer Edge.Cuts) (width 0.12))
   )
-  (module kbd:SW_Hole (layer F.Cu)
+  (module "my library:SW_Hole" (layer F.Cu)
     (at 57.15 47.625)
     (fp_text reference SW1 (at 4.6 6 180) (layer Dwgs.User) hide
